File: pcb/flyback.sch (KiCad schematic (older format))
At the start: 11 parts

Commit message: sync
Parts:
- removed 2000falan: R, symbol R
- removed C?: 0.01µ, symbol C
- removed C?: 0.1µ, symbol C
- removed R?: 10000, symbol R
- removed R?: 3000, symbol R
- removed R?: 100, symbol R
- removed R?: 1000, symbol R
- removed R?: 2400, symbol R
- removed U? (x2): LM358, symbol LM358
- removed U?: TLP250, Housings_DIP:DIP-8_W7.62mm, symbol TLP250
- added 10kpot1: POT, Potentiometers:Potentiometer_Alps_RK163_Single_Vertical, symbol POT
- added Cap1: C, Capacitors_THT:C_Rect_L9.0mm_W2.5mm_P7.50mm_MKT, symbol C
- added Csnub1: C, Capacitors_THT:CP_Radial_D7.5mm_P2.50mm, symbol C
- added Csnub2: C, Capacitors_THT:CP_Radial_D26.0mm_P10.00mm_SnapIn, symbol C
- added Dleft1, Dright1: D, Diodes_THT:D_DO-201AD_P12.70mm_Horizontal, symbol D
- added Dout1: D, Diodes_THT:D_5KPW_P12.70mm_Horizontal, symbol D
- added Dsnub1: D, Diodes_THT:D_A-405_P12.70mm_Horizontal, symbol D
- added Q1: IRF540N, TO_SOT_Packages_THT:TO-220-3_Vertical, symbol IRF540N
- added R1000falan1, R2200, R3000, Rload1: R, Resistors_THT:R_Axial_DIN0414_L11.9mm_D4.5mm_P15.24mm_Horizontal, symbol R
- added R93.44: R, Resistors_THT:R_Axial_Power_L38.0mm_W9.0mm_P45.72mm, symbol R
- added U1: LM358, Housings_DIP:DIP-8_W8.89mm_SMDSocket_LongPads, symbol LM358
- added tlpabimiz1: TLP250, Housings_DIP:DIP-8_W8.89mm_SMDSocket_LongPads, symbol TLP250
Connections:
- net +12V: now also U1.8 (V+), tlpabimiz1.8 (VCC)
- net -12VA: now also U1.4 (V-)
- net Earth: now also Cap1.2, Q1.3 (S), R2200.2, tlpabimiz1.3 (C), tlpabimiz1.5 (VEE)
- new net: Cap1.1, Dleft1.1 (K), Dright1.2 (A), U1.2 (-)
- new net: 10kpot1.1, Dleft1.2 (A)
- new net: 10kpot1.3, Dright1.1 (K)
- new net: 10kpot1.2, R1000falan1.2, R3000.1, U1.1
- new net: R2200.1, R3000.2, U1.3 (+)
- new net: R1000falan1.1, tlpabimiz1.2 (A)
- new net: Q1.1 (G), tlpabimiz1.6 (VO), tlpabimiz1.7 (VO)
- new net: Dsnub1.2 (A), Q1.2 (D)
- new net: Csnub1.2, Dsnub1.1 (K), R93.44.2
- new net: Csnub1.1, R93.44.1
- new net: Csnub2.1, Dout1.1 (K), Rload1.1
- new net: Csnub2.2, Rload1.2
